Commit message: worksheet2

File: rdl_turtlebot3_description/urdf/turtlebot3_simplified_burger.gazebo.xacro (robot description, xacro)
@@ -35,5 +35,5 @@
     <material>Gazebo/FlatBlack</material>
   </gazebo>
-  <gazebo>
+  <!--gazebo>
     <plugin name="turtlebot3_burger_controller" filename="libgazebo_ros_diff_drive.so">
       <commandTopic>cmd_vel</commandTopic>
@@ -55,4 +55,10 @@
       <wheelTorque>10</wheelTorque>
       <rosDebugLevel>na</rosDebugLevel>
+    </plugin>
+  </gazebo-->
+  <!-- ROS Control plugin for Gazebo -->
+  <gazebo>
+    <plugin name="gazebo_ros_control" filename="libgazebo_ros_control.so">
+      <robotNamespace>/turtlebot3_burger</robotNamespace>
     </plugin>
   </gazebo>

File: rdl_turtlebot3_description/urdf/turtlebot3_simplified_burger.urdf.xacro (robot description, xacro)
@@ -105,4 +105,26 @@
     <origin xyz="-0.081 0 -0.004" rpy="-1.57 0 0"/>
   </joint>
+  <!-- tag required by ros control for individual joint control -->
+  <transmission name="wheel_left_tran">
+    <type>transmission_interface/SimpleTransmission</type>
+    <joint name="wheel_left_joint">
+      <hardwareInterface>hardware_interface/EffortJointInterface</hardwareInterface>
+    </joint>
+    <actuator name="wheel_left">
+      <hardwareInterface>hardware_interface/EffortJointInterface</hardwareInterface>
+      <mechanicalReduction>1</mechanicalReduction>
+    </actuator>
+  </transmission>
+  <!-- tag required by ros control for individual joint control -->
+  <transmission name="wheel_right_tran">
+    <type>transmission_interface/SimpleTransmission</type>
+    <joint name="wheel_right_joint">
+      <hardwareInterface>hardware_interface/EffortJointInterface</hardwareInterface>
+    </joint>
+    <actuator name="wheel_right">
+      <hardwareInterface>hardware_interface/EffortJointInterface</hardwareInterface>
+      <mechanicalReduction>1</mechanicalReduction>
+    </actuator>
+  </transmission>
   <link name="caster_back_link">
     <collision>
